File: Boards/IRtransmitter/IRTransmitter.brd (EAGLE design)
At the start: 78.5 x 49 mm, 14 parts, among them IC1 MEGA8-P, Q1 BSS138

Commit message: schematic of IR receiver
Parts:
- added U$1: (no value), synergia_logo:SYNERGIA_30MM
Other:
- board text added: "J. Trzyna"
- board text added: "M. Trojan"
Changed lines of the file:
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@@
 <dimension x1="-6.5" y1="44.5" x2="-6.5" y2="-4.5" x3="-12.065" y3="20" textsize="1.778" layer="1"/>
 <dimension x1="-6.5" y1="-4.5" x2="72" y2="-4.5" x3="32.75" y3="-10.795" textsize="1.778" layer="1"/>
+<text x="60.96" y="8.255" size="1.778" layer="16" rot="MR0">J. Trzyna</text>
+<text x="60.96" y="4.445" size="1.778" layer="16" rot="MR0">M. Trojan</text>
 </plain>
 <attributes>
@@
 <element name="R6" library="rcl" package="R0805" value="1k" x="21.59" y="29.21" rot="MR90"/>
 <element name="R7" library="rcl" package="R0805" value="1k" x="19.05" y="29.21" rot="MR90"/>
+<element name="U$1" library="synergia_logo" package="SYNERGIA_30MM" value="" x="3.175" y="4.445" rot="MR90"/>
 </elements>
 <signals>
